File: 04_PROJECT/HybridPanda/HybridPanda.kicad_sch (KiCad schematic)
At the start: 114 parts, among them J1 SWD, P1 TYPE-C-31-M-04, Q1 DDTA143ECA-7-F P08, Q2 DDTA143ECA-7-F P08, Q3 PDTC114EU, Q4 HY12P03C2, SW1 SW_Push, U1 AP22615AWU-7, U10 TJA1042TK-3, U11 TJA1042TK-3, U12 XL1509-3.3, U3 10_0_QHHTZB6_3, U5 FM-B1921RGBA-SH, U6 TPS5450DDAR, U7 STM32H725ZGT6, U8 TJA1042TK-3, U9 TJA1042TK-3, Y1 25MHz X322525MOB4SI

Commit message: pcb: step 1 - apply footprint audit fixes (Q1/Q2/Q3 pads, U5, U12 EP, P1 ring, R6 R_0603, SMD attrs, 3D)
- Q3 SOT-323 pads to KiCad geometry; Q1/Q2 SOT-23 pads 0.6x1.475 + courtyard 3.1x3.5
- U5 LED pads y +/-0.60 per FM-B1921RGBA-SH datasheet
- U12 XL1509: EP pads lose paste/mask (SOP-8 without EP), SOIC-8 3D model
- P1 TYPE-C: THT pads B1-B12 0.60 -> 0.65, 12 stray F.Paste circles removed
- footprint attribute THT -> SMD on D1, D5-D9, Q1, Q2, U5, L3; L3 courtyard 8.9x6.8
- 3D models for D8/D9 (SOT-23) and Q4 (PowerPAK SO-8 step)
- R6 footprint Capacitor_SMD:C_0603 -> Resistor_SMD:R_0603 (schematic + board, nets kept)
- local reroute: relay_SBU1 via moved out of Q1 pad 3, R24 -0.35 mm, LED_RED nudged
- DRC 0 clearance / 0 unconnected / 181 (182 -> 181: -10 footprint_type, +10 lib mismatch, -1 text)
- new helpers 05_SCRIPTS/corr_gate.py, corr_step1_footprints.py, corr_step1b_fix.py, tools/dump_geom.py

Co-authored-by: Copilot <223556219+Copilot@users.noreply.github.com>
Parts:
- R6: footprint Capacitor_SMD:C_0603_1608Metric -> Resistor_SMD:R_0603_1608Metric

Commit message: Step 2: PCR-2 VFBSMPS-VCAP link, C64/C65 decoupling, PCR-1 PF9 solder jumper
Schematic: VFBSMPS global labels renamed to VCAP (ST AN5419 direct-SMPS
topology, VFBSMPS tied to VCAP; L5 2.2uH + C41/C42 kept on VLXSMPS/VCAP).
Added C64 2.2uF 0402 at VCAP pin 103, C65 4.7uF 0603 at VDDSMPS pin 16.
PCR-1: PF9 (HW_TYPE id1 bit 2) lifted from the GND strap and wired to JP1
(SolderJumper_2_Open, net Net-(JP1-B)); JP1 closed = RED (id1=0), open =
HYBRID (id1=4). ERC 0 errors.

PCB (05_SCRIPTS/corr_step2_pcb.py): net merge, PF7/PF8/PF10 GND straps
rebuilt, PF9 via + F.Cu track to JP1 (F.Cu 107.6,72.9), C65 on F.Cu
(109.3,70.1) 2.5 mm from pin 16, C64 on B.Cu (116.28,44.0) 1.5 mm from
pad 103 (SWDIO via moved 0.15 mm, C54 slid 0.15 mm east, pad 104 stub via
removed - pad stays on the B.Cu GND zone), VCAP link C42.1 -> via
(110.725,72.752) -> In1 13.9 mm -> existing VCAP In1 copper, 0.3 mm wide.
parity profile: PF9 expect float_or_low (JP1 strap).

Gates: DRC 0 clearance / 0 unconnected, 184 total (starved_thermal 17->18:
U7 pad 104), step7_validate no failures, final_audit shorts 0 / vip 0, ERC
0 errors.

Co-authored-by: Copilot <223556219+Copilot@users.noreply.github.com>
Parts:
- added C64: 2.2uF, Capacitor_SMD:C_0402_1005Metric, symbol Device:C_Small
- added C65: 4.7uF, Capacitor_SMD:C_0603_1608Metric, symbol Device:C_Small
- added JP1: HW_ID1, Jumper:SolderJumper-2_P1.3mm_Open_Pad1.0x1.5mm, symbol Jumper:SolderJumper_2_Open
Connections:
- net VFBSMPS is gone; now on net VCAP: C42.1, L5.2, U7.17 (VFBSMPS)
- net +3V3: now also C65.1
- net GND: now also C64.2, C65.2, JP1.1 (A); no longer U7.23 (PF9)
- net VCAP: now also C64.1
- new net: JP1.2 (B), U7.23 (PF9)
Other:
- note added: "PCR-1: JP1 fechado = RED (id1=0); aberto = HYBRID (id1=4)"
- note added: "PCR-2: VFBSMPS ligado a VCAP (AN5419 direct SMPS)"

Commit message: pcb: step 3 WIP - SI/PI HIGH items on schematic and PCB (DRC 0/0)
Schematic: R1 10k 0603, D15 BZT52C12 Vgs clamp, C4/C12 10uF, U13 USBLC6-2SC6.
PCB: R1/D15 rebuilt around the Q4 gate, R20/R21 moved next to U7 pads 100/101,
coupled In1 USB pair to U13 at U3, +5V feed to U1 widened. DRC: 0 clearance,
0 unconnected, 180 total (+1 silk_over_copper). See 06_REPORTS/corr/RESUME_STEP3.md.

Co-authored-by: Copilot <223556219+Copilot@users.noreply.github.com>
Parts:
- added D15: BZT52C12, Diode_SMD:D_SOD-123, symbol Device:D_Zener
- added U13: USBLC6-2SC6, Package_TO_SOT_SMD:SOT-23-6, symbol Power_Protection:USBLC6-2P6
- C12, C4: value 2.2uF -> 10uF; footprint Capacitor_SMD:C_0805_2012Metric -> Capacitor_SMD:C_1206_3216Metric
- R1: value 1K -> 10k; footprint Resistor_SMD:R_0402_1005Metric -> Resistor_SMD:R_0603_1608Metric
Connections:
- net 12V_Protected: now also D15.1 (K)
- net GND: now also U13.2 (GND)
- net USB_PWR: now also U13.5 (VBUS)
- net USB_R_D+: now also U13.3 (I/O2), U13.4 (I/O2)
- net USB_R_D-: now also U13.1 (I/O1), U13.6 (I/O1)
- net at D2.2 (A), Q4.4 (G), R1.2: now also D15.2 (A)
Other:
- note added: "Item 5 SI/PI: D15 zener 12 V limita Vgs de Q4 (K = 12V_Protected, A = gate)"
- note added: "Item 8 SI/PI: U13 ESD array USB (flow-through: lado conector pinos 1/3, lado MCU pinos 6/4)"

Commit message: pcb: step 3 - SI/PI HIGH items closed (C4/C12 0805 parity, U13 GND crossing fix, item 16 deferred)
Co-authored-by: Copilot <223556219+Copilot@users.noreply.github.com>
Parts:
- C12, C4: footprint Capacitor_SMD:C_1206_3216Metric -> Capacitor_SMD:C_0805_2012Metric

Commit message: pcb: step 4 - BOM impact of steps 1-3 (C4/C12 10uF, R1 10k 0603, C64/C65, D15, U13, R6 footprint; MPN/LCSC fields in schematic)
Co-authored-by: Copilot <223556219+Copilot@users.noreply.github.com>
Parts:
- C1, C11, C14, C2, C26, C27, C28, C29, C30, C31, C32, C33, C34, C38, C44, C45, C46, C47, C48, C49, C5, C50, C51, C52, C53, C54, C55, C56, C57, C58, C59: LCSC (none) -> C307331; MPN (none) -> CL05B104KB54PNC; Manufacturer (none) -> Samsung
- C10, C16, C17, C18, C19, C20, C21, C3: LCSC (none) -> C178332; MPN (none) -> 0805X476M100NT; Manufacturer (none) -> Fenghua
- C12, C4: LCSC (none) -> C2932476; MPN (none) -> CL21A106KBYQNNE; Manufacturer (none) -> Samsung
- C23, C24: LCSC (none) -> C1548; MPN (none) -> 0402CG150J500NT; Manufacturer (none) -> Fenghua
- C37: LCSC (none) -> C15195; MPN (none) -> CL05B103KB5NNNC; Manufacturer (none) -> Samsung
- C39, C40: LCSC (none) -> C23630; MPN (none) -> CL10A225KO8NNNC; Manufacturer (none) -> Samsung
- C41: LCSC (none) -> C1530; MPN (none) -> 0402B221K500NT; Manufacturer (none) -> Fenghua
- C42: LCSC (none) -> C15850; MPN (none) -> CL21A106KAYNNNE; Manufacturer (none) -> Samsung
- C43, C63: LCSC (none) -> C52923; MPN (none) -> CL05A105KA5NQNC; Manufacturer (none) -> Samsung
- C6, C7: LCSC (none) -> C125847; MPN (none) -> CC0805KKX7R9BB225; Manufacturer (none) -> Yageo
- C60, C61, C62, C65: LCSC (none) -> C19666; MPN (none) -> CL10A475KO8NNNC; Manufacturer (none) -> Samsung
- C64: LCSC (none) -> C23733; MPN (none) -> CL05A225MP5NSNC; Manufacturer (none) -> Samsung
- C8: LCSC (none) -> C315248; MPN (none) -> CL05A106MP5NUNC; Manufacturer (none) -> Samsung
- D1: LCSC (none) -> C148217; MPN (none) -> SMAJ16CA; Manufacturer (none) -> Littelfuse
- D10: LCSC (none) -> C426766; MPN (none) -> BAS70H,115; Manufacturer (none) -> Nexperia
- D11: LCSC (none) -> C85098; MPN (none) -> B340A-13-F; Manufacturer (none) -> Diodes Inc
- D12: LCSC (none) -> C72264; MPN (none) -> B540C-13-F; Manufacturer (none) -> Diodes Inc
- D13, D14: LCSC (none) -> C47546; MPN (none) -> BAT54S,215; Manufacturer (none) -> Nexperia
- D15: LCSC (none) -> C571379; MPN (none) -> BZT52C12; Manufacturer (none) -> High Diode (ou equivalente)
- D2: LCSC (none) -> C22648; MPN (none) -> BAS40WS 43; Manufacturer (none) -> Changjing
- D5, D6, D7, D8, D9: LCSC (none) -> C75176; MPN (none) -> PESD2CAN,215; Manufacturer (none) -> Nexperia
- FB1: LCSC (none) -> C1002; MPN (none) -> GZ1608D601TF; Manufacturer (none) -> Sunlord
- J1: LCSC (none) -> C150517; MPN (none) -> 20021121-00010C4LF; Manufacturer (none) -> Amphenol ICC
- L3: LCSC (none) -> C149588; MPN (none) -> SMMS0650-470M; Manufacturer (none) -> SXN
- L4: LCSC (none) -> C151872; MPN (none) -> MWSA1004S-150MT; Manufacturer (none) -> Sunlord
- L5: LCSC (none) -> C337891; MPN (none) -> DFE201610E-2R2M=P2; Manufacturer (none) -> Murata
- P1: MPN (none) -> TYPE-C-31-M-04; Manufacturer (none) -> Korean Hroparts
- Q1, Q2: LCSC (none) -> C460029; MPN (none) -> DDTA143ECA-7-F; Manufacturer (none) -> Diodes Inc
- Q3: LCSC (none) -> C135830; MPN (none) -> PDTC114EU,115; Manufacturer (none) -> Nexperia
- Q4: LCSC (none) -> C358006; MPN (none) -> HY12P03C2; Manufacturer (none) -> HUAYI
- R1: LCSC (none) -> C25804; MPN (none) -> 0603WAF1002T5E; Manufacturer (none) -> Uniroyal
- R14, R15, R16, R23, R24, R26, R28, R29, R3, R30, R31, R32, R33, R5, R9: LCSC (none) -> C25744; MPN (none) -> 0402WGF1002TCE; Manufacturer (none) -> Uniroyal
- R17: LCSC (none) -> C38941; MPN (none) -> 0402WGF1800TCE; Manufacturer (none) -> Uniroyal
- R18: LCSC (none) -> C413064; MPN (none) -> ERJ2RKF1100X; Manufacturer (none) -> Panasonic
- R19: LCSC (none) -> C25076; MPN (none) -> 0402WGF1000TCE; Manufacturer (none) -> Uniroyal
- R2: LCSC (none) -> C11702; MPN (none) -> 0402WGF1001TCE; Manufacturer (none) -> Uniroyal
- R20, R21: LCSC (none) -> C25092; MPN (none) -> 0402WGF220JTCE; Manufacturer (none) -> Uniroyal
- R27: LCSC (none) -> C25882; MPN (none) -> 0402WGF2401TCE; Manufacturer (none) -> Uniroyal
- R6: LCSC (none) -> C22993; MPN (none) -> 0603WAF3161T5E; Manufacturer (none) -> Uniroyal
- SW1: LCSC (none) -> C202424; MPN (none) -> SKQGAFE010; Manufacturer (none) -> Alps Alpine
- U1: MPN (none) -> AP22615AWU-7; Manufacturer (none) -> Diodes Inc
- U10, U11, U8, U9: LCSC (none) -> C131480; MPN (none) -> TJA1042TK/3/1J; Manufacturer (none) -> NXP
- U12: LCSC (none) -> C74193; MPN (none) -> XL1509-3.3E1; Manufacturer (none) -> XLSEMI
- U13: LCSC (none) -> C7519; MPN (none) -> USBLC6-2SC6; Manufacturer (none) -> STMicroelectronics
- U3: MPN (none) -> 10.0 QHHTZB6.3; Manufacturer (none) -> SHOU HAN
- U5: MPN (none) -> FM-B1921RGBA-SH; Manufacturer (none) -> Foshan NationStar
- U6: LCSC (none) -> C114425; MPN (none) -> TPS5450DDAR; Manufacturer (none) -> Texas Instruments
- U7: LCSC (none) -> C730156; MPN (none) -> STM32H725ZGT6; Manufacturer (none) -> STMicroelectronics
- Y1: LCSC (none) -> C9006; MPN (none) -> X322525MOB4SI; Manufacturer (none) -> YXC

Commit message: pcb: step 5 - SI/PI MEDIUM items (CAN 0.25, GND zone thermals, vias 0.6, stitching, outline +0.4, C23/C24 18pF, U3 shell GND)
Applied items 24, 26 (partial), 28, 30, 31, 33a/33b, 35 (partial), 12/13/14 (partial),
17 (partial), 20; each change gated by kicad-cli DRC (06_REPORTS/corr/drc_step5*.json).
DRC: 135 total, 0 clearance, 0 unconnected, 0 parity. ERC: 0 errors.
Deferred: 9, 16, 21-23, 25, 27, 29, 32, 34, 36 (see 06_REPORTS/corr/RESUME_STEP3.md).
final_audit.py: BOM MPN finding now data-driven; os._exit avoids pcbnew teardown hang.

Co-authored-by: Copilot <223556219+Copilot@users.noreply.github.com>
Parts:
- C23, C24: value 15pF -> 18pF; LCSC C1548 -> C1555; MPN 0402CG150J500NT -> 0402CG180J500NT
Connections:
- net GND: now also U3.5, U3.6
- no-connect marks 79 -> 77
